Commit message: Added extrinsic calibration override support for sensor URDF frames
Signed-off-by: Daun Jeong <jdu@robotis.com>

File: antbot_description/urdf/antbot.xacro (robot description, xacro)
@@ -9,4 +9,7 @@
   <xacro:include filename="$(find antbot_description)/urdf/wheel.xacro"/>
   <xacro:include filename="$(find antbot_description)/urdf/ros2_control.xacro"/>
+  <xacro:arg name="calibration_yaml_path" default=""/>
+  <xacro:property name="calibration_yaml_path_val" value="$(arg calibration_yaml_path)"/>
+  <xacro:property name="calibration_config" value="${xacro.load_yaml(calibration_yaml_path_val) if calibration_yaml_path_val != '' else dict()}"/>
   <!-- Wheel parameters -->
   <xacro:property name="wheelbase_length" value="0.530"/>
@@ -33,9 +36,15 @@
   <xacro:OpticalFrame name="camera_stereo_front_rgb_optical" parent="camera_stereo_front_rgb"/>
   <!-- Mono cameras -->
-  <xacro:Sensors name="camera_mono_left" xyz="0.260 0.25477 0.5875" rpy="0.0 0.0 ${radians(90)}"/>
+  <xacro:CalibratedSensors name="camera_mono_left"
+    default_xyz="0.260 0.25477 0.5875" default_rpy="0.0 0.0 ${radians(90)}"
+    calibration_key="camera_left_extrinsic"/>
   <xacro:OpticalFrame name="camera_mono_left_optical" parent="camera_mono_left"/>
-  <xacro:Sensors name="camera_mono_front" xyz="0.35807 0.0 0.5875" rpy="0.0 0.0 0.0"/>
+  <xacro:CalibratedSensors name="camera_mono_front"
+    default_xyz="0.35807 0.0 0.5875" default_rpy="0.0 0.0 0.0"
+    calibration_key="camera_front_extrinsic"/>
   <xacro:OpticalFrame name="camera_mono_front_optical" parent="camera_mono_front"/>
-  <xacro:Sensors name="camera_mono_right" xyz="0.260 -0.25477 0.5875" rpy="0.0 0.0 ${radians(-90)}"/>
+  <xacro:CalibratedSensors name="camera_mono_right"
+    default_xyz="0.260 -0.25477 0.5875" default_rpy="0.0 0.0 ${radians(-90)}"
+    calibration_key="camera_right_extrinsic"/>
   <xacro:OpticalFrame name="camera_mono_right_optical" parent="camera_mono_right"/>
   <xacro:Sensors name="camera_mono_back" xyz="-0.37669 0.0 0.299" rpy="0.0 0.0 ${radians(180)}"/>
@@ -49,5 +58,7 @@
   <xacro:Sensors name="lidar_2d_back" xyz="-0.325 0.0 0.255" rpy="${radians(180)} 0.0 0.0"/>
   <!-- 3D LiDAR -->
-  <xacro:Sensors name="lidar_3d" xyz="0.225332 0.0 0.724904" rpy="0.0 ${radians(10)} 0.0"/>
+  <xacro:CalibratedSensors name="lidar_3d"
+    default_xyz="0.225332 0.0 0.724904" default_rpy="0.0 ${radians(10)} 0.0"
+    calibration_key="lidar_3d_extrinsic"/>
   <xacro:SensorsRel parent="lidar_3d" child="lidar_3d_imu" xyz="0.00677 -0.02045 -0.02597" rpy="0.0 0.0 0.0"/>
   <!-- Charging coil -->

File: antbot_description/urdf/sensors.xacro (robot description, xacro)
@@ -29,3 +29,18 @@
     <link name="${name}_link"/>
   </xacro:macro>
+  <xacro:macro name="CalibratedSensors" params="name default_xyz default_rpy calibration_key">
+    <xacro:property name="calib_data" value="${calibration_config.get(calibration_key)}"/>
+    <xacro:property name="_xyz" value="${
+      str(calib_data['tx']) + ' ' + str(calib_data['ty']) + ' ' + str(calib_data['tz'])
+      if calib_data else default_xyz}"/>
+    <xacro:property name="_rpy" value="${
+      str(calib_data['rx']) + ' ' + str(calib_data['ry']) + ' ' + str(calib_data['rz'])
+      if calib_data else default_rpy}"/>
+    <joint name="${name}_joint" type="fixed">
+      <parent link="base_link"/>
+      <child link="${name}_link"/>
+      <origin xyz="${_xyz}" rpy="${_rpy}"/>
+    </joint>
+    <link name="${name}_link"/>
+  </xacro:macro>
 </robot>

Commit message: Restructured urdf
Signed-off-by: Daun Jeong <jdu@robotis.com>

File: antbot_description/urdf/antbot.xacro (robot description, xacro)
@@ -2,71 +2,155 @@
 <!--
   Main URDF for ANTBot swerve-drive delivery robot.
-  Based on G50 hardware platform.
+  G50 hardware platform based 4-wheel independent steering (swerve-drive) mobile base.
+  Assembles:
+    - Base body (base_link + body_link)
+    - 4 swerve wheel modules
+    - All sensors (cameras, IMU, GNSS, magnetometer, LiDARs)
+    - Miscellaneous frames (charging coil)
+    - ros2_control hardware interface for the base platform
 -->
 <robot name="antbot" xmlns:xacro="http://ros.org/wiki/xacro">
-  <xacro:include filename="$(find antbot_description)/urdf/sensors.xacro"/>
-  <xacro:include filename="$(find antbot_description)/urdf/base.xacro"/>
-  <xacro:include filename="$(find antbot_description)/urdf/wheel.xacro"/>
+  <!-- ============================================================
+       Include: ANTBot module files
+       ============================================================ -->
+  <xacro:include filename="$(find antbot_description)/urdf/base_body.xacro"/>
+  <xacro:include filename="$(find antbot_description)/urdf/drive/wheel_module.xacro"/>
+  <xacro:include filename="$(find antbot_description)/urdf/sensor/common.xacro"/>
+  <xacro:include filename="$(find antbot_description)/urdf/sensor/depth_camera.xacro"/>
+  <xacro:include filename="$(find antbot_description)/urdf/sensor/mono_camera.xacro"/>
+  <xacro:include filename="$(find antbot_description)/urdf/sensor/imu.xacro"/>
+  <xacro:include filename="$(find antbot_description)/urdf/sensor/lidar_2d.xacro"/>
+  <xacro:include filename="$(find antbot_description)/urdf/sensor/lidar_3d.xacro"/>
   <xacro:include filename="$(find antbot_description)/urdf/ros2_control.xacro"/>
+  <!-- ============================================================
+       Calibration YAML loading
+       If calibration_yaml_path is passed, values loaded here are consumed
+       by CalibratedSensorFrame (see sensor/common.xacro).
+       ============================================================ -->
   <xacro:arg name="calibration_yaml_path" default=""/>
   <xacro:property name="calibration_yaml_path_val" value="$(arg calibration_yaml_path)"/>
   <xacro:property name="calibration_config" value="${xacro.load_yaml(calibration_yaml_path_val) if calibration_yaml_path_val != '' else dict()}"/>
-  <!-- Wheel parameters -->
-  <xacro:property name="wheelbase_length" value="0.530"/>
-  <xacro:property name="wheelbase_width" value="0.512"/>
-  <xacro:property name="steering_width" value="0.401"/>
-  <xacro:property name="wheel_radius" value="0.103"/>
-  <xacro:property name="steering_height" value="0.120"/>
-  <xacro:property name="wheel_offset" value="${(wheelbase_width - steering_width)/2}"/>
-  <!-- Base body assembly -->
-  <xacro:Base/>
-  <!-- Swerve drive wheel system -->
-  <xacro:SwerveWheelLeft position_name="front_left"
-                         x_pos="${wheelbase_length/2}" y_pos="${steering_width/2}"/>
-  <xacro:SwerveWheelRight position_name="front_right"
-                          x_pos="${wheelbase_length/2}" y_pos="${-steering_width/2}"/>
-  <xacro:SwerveWheelLeft position_name="rear_left"
-                         x_pos="${-wheelbase_length/2}" y_pos="${steering_width/2}"/>
-  <xacro:SwerveWheelRight position_name="rear_right"
-                          x_pos="${-wheelbase_length/2}" y_pos="${-steering_width/2}"/>
-  <!-- Stereo cameras -->
-  <xacro:Sensors name="camera_stereo_front_depth" xyz="0.348162 0.0475 0.526484" rpy="0.0 ${radians(30)} 0.0"/>
-  <xacro:OpticalFrame name="camera_stereo_front_depth_optical" parent="camera_stereo_front_depth"/>
-  <xacro:SensorsRel parent="camera_stereo_front_depth" child="camera_stereo_front_rgb" xyz="0.0 -0.124 0.0" rpy="0.0 0.0 0.0"/>
-  <xacro:OpticalFrame name="camera_stereo_front_rgb_optical" parent="camera_stereo_front_rgb"/>
-  <!-- Mono cameras -->
-  <xacro:CalibratedSensors name="camera_mono_left"
-    default_xyz="0.260 0.25477 0.5875" default_rpy="0.0 0.0 ${radians(90)}"
+  <!-- ============================================================
+       Robot dimension properties
+       ============================================================ -->
+  <xacro:property name="wheel_radius"     value="0.103"/>  <!-- Wheel radius [m] -->
+  <xacro:property name="base_link_height" value="0.103"/>  <!-- Height from base_link (ground) to body_link [m] (= wheel_radius) -->
+  <xacro:property name="wheelbase_length" value="0.530"/>  <!-- X-axis distance between front/rear wheels [m] -->
+  <xacro:property name="steering_width"   value="0.401"/>  <!-- Y-axis distance between left/right steering axes [m] -->
+  <xacro:property name="wheel_offset"     value="0.055"/>  <!-- Y-axis offset from steering axis to wheel center [m] -->
+  <!-- ============================================================
+       Material definitions
+       ============================================================ -->
+  <material name="white">
+    <color rgba="1.0 1.0 1.0 1.0"/>
+  </material>
+  <material name="black">
+    <color rgba="0.2 0.2 0.2 1.0"/>
+  </material>
+  <material name="gray">
+    <color rgba="0.5 0.5 0.5 1.0"/>
+  </material>
+  <!-- ============================================================
+       1. Base body assembly (base_link ground frame + body_link chassis)
+       ============================================================ -->
+  <xacro:BaseBody/>
+  <!-- ============================================================
+       2. Swerve wheel system (4-wheel independent steering)
+       Placement: front-left, front-right, rear-left, rear-right
+       ============================================================ -->
+  <xacro:SwerveWheel position_name="front_left"
+    x_pos="${wheelbase_length / 2}" y_pos="${steering_width / 2}" side="1"/>
+  <xacro:SwerveWheel position_name="front_right"
+    x_pos="${wheelbase_length / 2}" y_pos="${-steering_width / 2}" side="-1"/>
+  <xacro:SwerveWheel position_name="rear_left"
+    x_pos="${-wheelbase_length / 2}" y_pos="${steering_width / 2}" side="1"/>
+  <xacro:SwerveWheel position_name="rear_right"
+    x_pos="${-wheelbase_length / 2}" y_pos="${-steering_width / 2}" side="-1"/>
+  <!-- ============================================================
+       3. Sensor placement
+       Each sensor is registered by calling the corresponding module macro.
+       To add another instance of the same sensor, call the macro again
+       with a new position.
+       Sensors use body_link (chassis frame) as their parent. The z
+       values below are heights above body_link, pre-computed as
+       (ground-referenced height) - base_link_height (0.103 m).
+       ============================================================ -->
+  <!-- === Stereo depth camera (front top) === -->
+  <!-- z = 0.629484 - 0.103 = 0.526484 -->
+  <xacro:DepthCamera name="camera_stereo_front" parent="body_link"
+    xyz="0.348162 0.0475 0.526484"
+    rpy="0.0 ${radians(30)} 0.0"/>
+  <!-- === 4 mono cameras === -->
+  <!-- Left: 90° left-facing -->
+  <!-- z = 0.5875 - 0.103 = 0.4845 -->
+  <xacro:MonoCamera name="camera_mono_left" parent="body_link"
+    xyz="0.260 0.25477 0.4845"
+    rpy="0.0 0.0 ${radians(90)}"
     calibration_key="camera_left_extrinsic"/>
-  <xacro:OpticalFrame name="camera_mono_left_optical" parent="camera_mono_left"/>
-  <xacro:CalibratedSensors name="camera_mono_front"
-    default_xyz="0.35807 0.0 0.5875" default_rpy="0.0 0.0 0.0"
+  <!-- Front: forward-facing -->
+  <!-- z = 0.5875 - 0.103 = 0.4845 -->
+  <xacro:MonoCamera name="camera_mono_front" parent="body_link"
+    xyz="0.35807 0.0 0.4845"
+    rpy="0.0 0.0 0.0"
     calibration_key="camera_front_extrinsic"/>
-  <xacro:OpticalFrame name="camera_mono_front_optical" parent="camera_mono_front"/>
-  <xacro:CalibratedSensors name="camera_mono_right"
-    default_xyz="0.260 -0.25477 0.5875" default_rpy="0.0 0.0 ${radians(-90)}"
+  <!-- Right: 90° right-facing -->
+  <!-- z = 0.5875 - 0.103 = 0.4845 -->
+  <xacro:MonoCamera name="camera_mono_right" parent="body_link"
+    xyz="0.260 -0.25477 0.4845"
+    rpy="0.0 0.0 ${radians(-90)}"
     calibration_key="camera_right_extrinsic"/>
-  <xacro:OpticalFrame name="camera_mono_right_optical" parent="camera_mono_right"/>
-  <xacro:Sensors name="camera_mono_back" xyz="-0.37669 0.0 0.299" rpy="0.0 0.0 ${radians(180)}"/>
-  <xacro:OpticalFrame name="camera_mono_back_optical" parent="camera_mono_back"/>
-  <!-- IMU / GNSS / Magnetometer -->
-  <xacro:Sensors name="imu" xyz="0.240 0.00675 0.3902" rpy="0.0 0.0 ${radians(180)}"/>
-  <xacro:Sensors name="gnss" xyz="0.2026 -0.128 0.660" rpy="0.0 0.0 ${radians(180)}"/>
-  <xacro:Sensors name="magnetometer" xyz="0.240 -0.00425 0.3902" rpy="0.0 0.0 0.0"/>
-  <!-- 2D LiDARs -->
-  <xacro:CalibratedSensors name="lidar_2d_front"
-    default_xyz="0.325 0.0 0.255" default_rpy="0.0 ${radians(180)} 0.0"
+  <!-- Rear: 180° backward-facing (no calibration) -->
+  <!-- z = 0.299 - 0.103 = 0.196 -->
+  <xacro:MonoCamera name="camera_mono_back" parent="body_link"
+    xyz="-0.37669 0.0 0.196"
+    rpy="0.0 0.0 ${radians(180)}"/>
+  <!-- === Inertial/navigation sensors === -->
+  <!-- z = 0.3902 - 0.103 = 0.2872 -->
+  <xacro:Imu name="imu" parent="body_link"
+    xyz="0.240 0.00675 0.2872"
+    rpy="0.0 0.0 ${radians(180)}"/>
+  <!-- z = 0.660 - 0.103 = 0.557 -->
+  <xacro:Gnss name="gnss" parent="body_link"
+    xyz="0.2026 -0.128 0.557"
+    rpy="0.0 0.0 ${radians(180)}"/>
+  <!-- z = 0.3902 - 0.103 = 0.2872 -->
+  <xacro:Magnetometer name="magnetometer" parent="body_link"
+    xyz="0.240 -0.00425 0.2872"
+    rpy="0.0 0.0 0.0"/>
+  <!-- === 2D LiDAR (front/rear) === -->
+  <!-- z = 0.255 - 0.103 = 0.152 -->
+  <xacro:Lidar2d name="lidar_2d_front" parent="body_link"
+    xyz="0.325 0.0 0.152"
+    rpy="0.0 ${radians(180)} 0.0"
     calibration_key="lidar_2d_front_extrinsic"/>
-  <xacro:CalibratedSensors name="lidar_2d_back"
-    default_xyz="-0.325 0.0 0.255" default_rpy="${radians(180)} 0.0 0.0"
+  <!-- z = 0.255 - 0.103 = 0.152 -->
+  <xacro:Lidar2d name="lidar_2d_back" parent="body_link"
+    xyz="-0.325 0.0 0.152"
+    rpy="${radians(180)} 0.0 0.0"
     calibration_key="lidar_2d_back_extrinsic"/>
-  <!-- 3D LiDAR -->
-  <xacro:CalibratedSensors name="lidar_3d"
-    default_xyz="0.225332 0.0 0.724904" default_rpy="0.0 ${radians(10)} 0.0"
+  <!-- === 3D LiDAR (top, 10° forward tilt) === -->
+  <!-- z = 0.724904 - 0.103 = 0.621904 -->
+  <xacro:Lidar3d name="lidar_3d" parent="body_link"
+    xyz="0.225332 0.0 0.621904"
+    rpy="0.0 ${radians(10)} 0.0"
     calibration_key="lidar_3d_extrinsic"/>
-  <xacro:SensorsRel parent="lidar_3d" child="lidar_3d_imu" xyz="0.00677 -0.02045 -0.02597" rpy="0.0 0.0 0.0"/>
-  <!-- Charging coil -->
-  <xacro:Sensors name="robot_charging_coil" xyz="-0.299119 0.0 0.170631" rpy="0.0 0.0 0.0"/>
-  <!-- ros2_control hardware interface -->
-  <xacro:antbot_ros2_control/>
+  <!-- ============================================================
+       4. Miscellaneous frames
+       ============================================================ -->
+  <!-- Charging coil: lower rear of robot, used for charging station alignment -->
+  <!-- z = 0.170631 - 0.103 = 0.067631 -->
+  <xacro:SensorFrame name="robot_charging_coil" parent="body_link"
+    xyz="-0.299119 0.0 0.067631"
+    rpy="0.0 0.0 0.0"/>
+  <!-- ============================================================
+       TODO: Accessories (cargo lid, flag pole) — attach to body_link
+       Add includes like:
+         <xacro:include filename="$(find antbot_description)/urdf/accessory/cargo_lid.xacro"/>
+         <xacro:include filename="$(find antbot_description)/urdf/accessory/flag_pole.xacro"/>
+       and the corresponding macro calls here.
+       ============================================================ -->
+  <!-- ============================================================
+       5. ros2_control hardware interface
+       ============================================================ -->
+  <xacro:AntbotRos2Control/>
 </robot>

File: antbot_description/urdf/ros2_control.xacro (robot description, xacro)
@@ -1,14 +1,18 @@
 <?xml version="1.0"?>
 <!--
-  ros2_control hardware interface definition for ANTBot.
-  Uses antbot/hw_interface/BoardInterface plugin.
+  ros2_control hardware interface definition for the base platform.
+  Controls 8 joints via the ANTBot BoardInterface plugin.
+  Joint configuration:
+    - 4 drive joints (wheel_*_joint):    velocity/acceleration command, velocity/position/effort feedback
+    - 4 steering joints (steering_*_joint): position/velocity/acceleration command, position/effort feedback
 -->
 <robot xmlns:xacro="http://www.ros.org/wiki/xacro">
-  <xacro:macro name="antbot_ros2_control">
-    <ros2_control name="ant_hardware" type="system">
+  <xacro:macro name="AntbotRos2Control">
+    <ros2_control name="base_hardware" type="system">
       <hardware>
         <plugin>antbot/hw_interface/BoardInterface</plugin>
       </hardware>
-      <!-- Wheel joints (velocity command) -->
+      <!-- === Drive (Wheel) joints: velocity control === -->
+      <!-- Controls each wheel's rotational velocity to drive the robot -->
       <joint name="wheel_front_left_joint">
         <command_interface name="velocity"/>
@@ -39,5 +43,6 @@
         <state_interface name="position"/>
       </joint>
-      <!-- Steering joints (position command) -->
+      <!-- === Steering joints: position control === -->
+      <!-- Controls each wheel's heading angle for steering -->
       <joint name="steering_front_left_joint">
         <command_interface name="position"/>

File: antbot_gazebo/urdf/antbot_sim.xacro (robot description, xacro)
@@ -52,4 +52,4 @@
   <xacro:Sensors name="robot_charging_coil" xyz="-0.299119 0.0 0.170631" rpy="0.0 0.0 0.0"/>
   <!-- Gazebo ros2_control -->
-  <xacro:antbot_ros2_control_gazebo/>
+  <xacro:AntbotRos2ControlGazebo/>
 </robot>

File: antbot_gazebo/urdf/ros2_control_gazebo.xacro (robot description, xacro)
@@ -1,6 +1,6 @@
 <?xml version="1.0"?>
 <robot xmlns:xacro="http://www.ros.org/wiki/xacro">
-  <xacro:macro name="antbot_ros2_control_gazebo">
-    <ros2_control name="ant_hardware" type="system">
+  <xacro:macro name="AntbotRos2ControlGazebo">
+    <ros2_control name="base_hardware" type="system">
       <hardware>
         <plugin>ign_ros2_control/IgnitionSystem</plugin>
