Commit message: Restructured URDF and fixed navigation map display
Signed-off-by: Daun Jeong <jdu@robotis.com>

File: antbot_description/urdf/antbot.xacro (robot description, xacro)
@@ -1,156 +1,13 @@
 <?xml version="1.0" ?>
 <!--
-  Main URDF for ANTBot swerve-drive delivery robot.
-  G50 hardware platform based 4-wheel independent steering (swerve-drive) mobile base.
-  Assembles:
-    - Base body (base_link + body_link)
-    - 4 swerve wheel modules
-    - All sensors (cameras, IMU, GNSS, magnetometer, LiDARs)
-    - Miscellaneous frames (charging coil)
-    - ros2_control hardware interface for the base platform
+  Top-level URDF for the real ANTBot hardware platform.
+  Combines the shared core (antbot_core.xacro) with the real-hardware
+  ros2_control interface (ros2_control.xacro).
+  For the Gazebo simulation variant, see antbot_gazebo/urdf/antbot_sim.xacro.
 -->
 <robot name="antbot" xmlns:xacro="http://ros.org/wiki/xacro">
-  <!-- ============================================================
-       Include: ANTBot module files
-       ============================================================ -->
-  <xacro:include filename="$(find antbot_description)/urdf/base_body.xacro"/>
-  <xacro:include filename="$(find antbot_description)/urdf/drive/wheel_module.xacro"/>
-  <xacro:include filename="$(find antbot_description)/urdf/sensor/common.xacro"/>
-  <xacro:include filename="$(find antbot_description)/urdf/sensor/depth_camera.xacro"/>
-  <xacro:include filename="$(find antbot_description)/urdf/sensor/mono_camera.xacro"/>
-  <xacro:include filename="$(find antbot_description)/urdf/sensor/imu.xacro"/>
-  <xacro:include filename="$(find antbot_description)/urdf/sensor/lidar_2d.xacro"/>
-  <xacro:include filename="$(find antbot_description)/urdf/sensor/lidar_3d.xacro"/>
+  <xacro:include filename="$(find antbot_description)/urdf/antbot_core.xacro"/>
   <xacro:include filename="$(find antbot_description)/urdf/ros2_control.xacro"/>
-  <!-- ============================================================
-       Calibration YAML loading
-       If calibration_yaml_path is passed, values loaded here are consumed
-       by CalibratedSensorFrame (see sensor/common.xacro).
-       ============================================================ -->
-  <xacro:arg name="calibration_yaml_path" default=""/>
-  <xacro:property name="calibration_yaml_path_val" value="$(arg calibration_yaml_path)"/>
-  <xacro:property name="calibration_config" value="${xacro.load_yaml(calibration_yaml_path_val) if calibration_yaml_path_val != '' else dict()}"/>
-  <!-- ============================================================
-       Robot dimension properties
-       ============================================================ -->
-  <xacro:property name="wheel_radius"     value="0.103"/>  <!-- Wheel radius [m] -->
-  <xacro:property name="base_link_height" value="0.103"/>  <!-- Height from base_link (ground) to body_link [m] (= wheel_radius) -->
-  <xacro:property name="wheelbase_length" value="0.530"/>  <!-- X-axis distance between front/rear wheels [m] -->
-  <xacro:property name="steering_width"   value="0.401"/>  <!-- Y-axis distance between left/right steering axes [m] -->
-  <xacro:property name="wheel_offset"     value="0.055"/>  <!-- Y-axis offset from steering axis to wheel center [m] -->
-  <!-- ============================================================
-       Material definitions
-       ============================================================ -->
-  <material name="white">
-    <color rgba="1.0 1.0 1.0 1.0"/>
-  </material>
-  <material name="black">
-    <color rgba="0.2 0.2 0.2 1.0"/>
-  </material>
-  <material name="gray">
-    <color rgba="0.5 0.5 0.5 1.0"/>
-  </material>
-  <!-- ============================================================
-       1. Base body assembly (base_link ground frame + body_link chassis)
-       ============================================================ -->
-  <xacro:BaseBody/>
-  <!-- ============================================================
-       2. Swerve wheel system (4-wheel independent steering)
-       Placement: front-left, front-right, rear-left, rear-right
-       ============================================================ -->
-  <xacro:SwerveWheel position_name="front_left"
-    x_pos="${wheelbase_length / 2}" y_pos="${steering_width / 2}" side="1"/>
-  <xacro:SwerveWheel position_name="front_right"
-    x_pos="${wheelbase_length / 2}" y_pos="${-steering_width / 2}" side="-1"/>
-  <xacro:SwerveWheel position_name="rear_left"
-    x_pos="${-wheelbase_length / 2}" y_pos="${steering_width / 2}" side="1"/>
-  <xacro:SwerveWheel position_name="rear_right"
-    x_pos="${-wheelbase_length / 2}" y_pos="${-steering_width / 2}" side="-1"/>
-  <!-- ============================================================
-       3. Sensor placement
-       Each sensor is registered by calling the corresponding module macro.
-       To add another instance of the same sensor, call the macro again
-       with a new position.
-       Sensors use body_link (chassis frame) as their parent. The z
-       values below are heights above body_link, pre-computed as
-       (ground-referenced height) - base_link_height (0.103 m).
-       ============================================================ -->
-  <!-- === Stereo depth camera (front top) === -->
-  <!-- z = 0.629484 - 0.103 = 0.526484 -->
-  <xacro:DepthCamera name="camera_stereo_front" parent="body_link"
-    xyz="0.348162 0.0475 0.526484"
-    rpy="0.0 ${radians(30)} 0.0"/>
-  <!-- === 4 mono cameras === -->
-  <!-- Left: 90° left-facing -->
-  <!-- z = 0.5875 - 0.103 = 0.4845 -->
-  <xacro:MonoCamera name="camera_mono_left" parent="body_link"
-    xyz="0.260 0.25477 0.4845"
-    rpy="0.0 0.0 ${radians(90)}"
-    calibration_key="camera_left_extrinsic"/>
-  <!-- Front: forward-facing -->
-  <!-- z = 0.5875 - 0.103 = 0.4845 -->
-  <xacro:MonoCamera name="camera_mono_front" parent="body_link"
-    xyz="0.35807 0.0 0.4845"
-    rpy="0.0 0.0 0.0"
-    calibration_key="camera_front_extrinsic"/>
-  <!-- Right: 90° right-facing -->
-  <!-- z = 0.5875 - 0.103 = 0.4845 -->
-  <xacro:MonoCamera name="camera_mono_right" parent="body_link"
-    xyz="0.260 -0.25477 0.4845"
-    rpy="0.0 0.0 ${radians(-90)}"
-    calibration_key="camera_right_extrinsic"/>
-  <!-- Rear: 180° backward-facing (no calibration) -->
-  <!-- z = 0.299 - 0.103 = 0.196 -->
-  <xacro:MonoCamera name="camera_mono_back" parent="body_link"
-    xyz="-0.37669 0.0 0.196"
-    rpy="0.0 0.0 ${radians(180)}"/>
-  <!-- === Inertial/navigation sensors === -->
-  <!-- z = 0.3902 - 0.103 = 0.2872 -->
-  <xacro:Imu name="imu" parent="body_link"
-    xyz="0.240 0.00675 0.2872"
-    rpy="0.0 0.0 ${radians(180)}"/>
-  <!-- z = 0.660 - 0.103 = 0.557 -->
-  <xacro:Gnss name="gnss" parent="body_link"
-    xyz="0.2026 -0.128 0.557"
-    rpy="0.0 0.0 ${radians(180)}"/>
-  <!-- z = 0.3902 - 0.103 = 0.2872 -->
-  <xacro:Magnetometer name="magnetometer" parent="body_link"
-    xyz="0.240 -0.00425 0.2872"
-    rpy="0.0 0.0 0.0"/>
-  <!-- === 2D LiDAR (front/rear) === -->
-  <!-- z = 0.255 - 0.103 = 0.152 -->
-  <xacro:Lidar2d name="lidar_2d_front" parent="body_link"
-    xyz="0.325 0.0 0.152"
-    rpy="0.0 ${radians(180)} 0.0"
-    calibration_key="lidar_2d_front_extrinsic"/>
-  <!-- z = 0.255 - 0.103 = 0.152 -->
-  <xacro:Lidar2d name="lidar_2d_back" parent="body_link"
-    xyz="-0.325 0.0 0.152"
-    rpy="${radians(180)} 0.0 0.0"
-    calibration_key="lidar_2d_back_extrinsic"/>
-  <!-- === 3D LiDAR (top, 10° forward tilt) === -->
-  <!-- z = 0.724904 - 0.103 = 0.621904 -->
-  <xacro:Lidar3d name="lidar_3d" parent="body_link"
-    xyz="0.225332 0.0 0.621904"
-    rpy="0.0 ${radians(10)} 0.0"
-    calibration_key="lidar_3d_extrinsic"/>
-  <!-- ============================================================
-       4. Miscellaneous frames
-       ============================================================ -->
-  <!-- Charging coil: lower rear of robot, used for charging station alignment -->
-  <!-- z = 0.170631 - 0.103 = 0.067631 -->
-  <xacro:SensorFrame name="robot_charging_coil" parent="body_link"
-    xyz="-0.299119 0.0 0.067631"
-    rpy="0.0 0.0 0.0"/>
-  <!-- ============================================================
-       TODO: Accessories (cargo lid, flag pole) — attach to body_link
-       Add includes like:
-         <xacro:include filename="$(find antbot_description)/urdf/accessory/cargo_lid.xacro"/>
-         <xacro:include filename="$(find antbot_description)/urdf/accessory/flag_pole.xacro"/>
-       and the corresponding macro calls here.
-       ============================================================ -->
-  <!-- ============================================================
-       5. ros2_control hardware interface
-       ============================================================ -->
+  <xacro:AntbotCore/>
   <xacro:AntbotRos2Control/>
 </robot>

File: antbot_gazebo/urdf/antbot_sim.xacro (robot description, xacro)
@@ -1,55 +1,14 @@
 <?xml version="1.0" ?>
+<!--
+  Top-level URDF for the ANTBot Gazebo simulation.
+  Combines the shared core (antbot_description/urdf/antbot_core.xacro) with
+  Gazebo-specific ros2_control (ign_ros2_control) and sensor plugins.
+  For the real-hardware variant, see antbot_description/urdf/antbot.xacro.
+-->
 <robot name="antbot" xmlns:xacro="http://ros.org/wiki/xacro">
-  <!-- Import shared macros from antbot_description -->
-  <xacro:include filename="$(find antbot_description)/urdf/sensors.xacro"/>
-  <xacro:include filename="$(find antbot_description)/urdf/base.xacro"/>
-  <xacro:include filename="$(find antbot_description)/urdf/wheel.xacro"/>
-  <!-- antbot_gazebo definitions -->
+  <xacro:include filename="$(find antbot_description)/urdf/antbot_core.xacro"/>
   <xacro:include filename="$(find antbot_gazebo)/urdf/ros2_control_gazebo.xacro"/>
   <xacro:include filename="$(find antbot_gazebo)/urdf/gazebo_plugins.xacro"/>
-  <!-- Wheel parameters -->
-  <xacro:property name="wheelbase_length" value="0.530"/>
-  <xacro:property name="wheelbase_width" value="0.512"/>
-  <xacro:property name="steering_width" value="0.401"/>
-  <xacro:property name="wheel_radius" value="0.103"/>
-  <xacro:property name="steering_height" value="0.120"/>
-  <xacro:property name="wheel_offset" value="${(wheelbase_width - steering_width)/2}"/>
-  <!-- Base body -->
-  <xacro:Base/>
-  <!-- 4 swerve wheels -->
-  <xacro:SwerveWheelLeft position_name="front_left"
-                         x_pos="${wheelbase_length/2}" y_pos="${steering_width/2}"/>
-  <xacro:SwerveWheelRight position_name="front_right"
-                          x_pos="${wheelbase_length/2}" y_pos="${-steering_width/2}"/>
-  <xacro:SwerveWheelLeft position_name="rear_left"
-                         x_pos="${-wheelbase_length/2}" y_pos="${steering_width/2}"/>
-  <xacro:SwerveWheelRight position_name="rear_right"
-                          x_pos="${-wheelbase_length/2}" y_pos="${-steering_width/2}"/>
-  <!-- Stereo camera -->
-  <xacro:Sensors name="camera_stereo_front_depth" xyz="0.348162 0.0475 0.526484" rpy="0.0 ${radians(30)} 0.0"/>
-  <xacro:OpticalFrame name="camera_stereo_front_depth_optical" parent="camera_stereo_front_depth"/>
-  <xacro:SensorsRel parent="camera_stereo_front_depth" child="camera_stereo_front_rgb" xyz="0.0 -0.124 0.0" rpy="0.0 0.0 0.0"/>
-  <xacro:OpticalFrame name="camera_stereo_front_rgb_optical" parent="camera_stereo_front_rgb"/>
-  <!-- Mono cameras -->
-  <xacro:Sensors name="camera_mono_left" xyz="0.260 0.25477 0.5875" rpy="0.0 0.0 ${radians(90)}"/>
-  <xacro:OpticalFrame name="camera_mono_left_optical" parent="camera_mono_left"/>
-  <xacro:Sensors name="camera_mono_front" xyz="0.35807 0.0 0.5875" rpy="0.0 0.0 0.0"/>
-  <xacro:OpticalFrame name="camera_mono_front_optical" parent="camera_mono_front"/>
-  <xacro:Sensors name="camera_mono_right" xyz="0.260 -0.25477 0.5875" rpy="0.0 0.0 ${radians(-90)}"/>
-  <xacro:OpticalFrame name="camera_mono_right_optical" parent="camera_mono_right"/>
-  <xacro:Sensors name="camera_mono_back" xyz="-0.37669 0.0 0.299" rpy="0.0 0.0 ${radians(180)}"/>
-  <xacro:OpticalFrame name="camera_mono_back_optical" parent="camera_mono_back"/>
-  <!-- IMU / GNSS / Magnetometer -->
-  <xacro:Sensors name="imu" xyz="0.240 0.00675 0.3902" rpy="0.0 0.0 ${radians(180)}"/>
-  <xacro:Sensors name="gnss" xyz="0.2026 -0.128 0.660" rpy="0.0 0.0 ${radians(180)}"/>
-  <xacro:Sensors name="magnetometer" xyz="0.240 -0.00425 0.3902" rpy="0.0 0.0 0.0"/>
-  <!-- 2D LiDAR -->
-  <xacro:Sensors name="lidar_2d_front" xyz="0.325 0.0 0.255" rpy="0.0 0.0 ${radians(180)}"/>
-  <xacro:Sensors name="lidar_2d_back" xyz="-0.325 0.0 0.255" rpy="0.0 0.0 0.0"/>
-  <!-- 3D LiDAR -->
-  <xacro:Sensors name="lidar_3d" xyz="0.225332 0.0 0.724904" rpy="0.0 ${radians(10)} 0.0"/>
-  <!-- Charging coil -->
-  <xacro:Sensors name="robot_charging_coil" xyz="-0.299119 0.0 0.170631" rpy="0.0 0.0 0.0"/>
-  <!-- Gazebo ros2_control -->
+  <xacro:AntbotCore/>
   <xacro:AntbotRos2ControlGazebo/>
 </robot>

File: antbot_gazebo/urdf/gazebo_plugins.xacro (robot description, xacro)
@@ -6,7 +6,9 @@
     <mu2>0.2</mu2>
   </gazebo>
-  <!-- ── Wheel friction macro ── -->
-  <xacro:macro name="WheelFriction" params="prefix">
-    <gazebo reference="${prefix}_wheel_link">
+  <!-- ── Wheel friction macro ──
+       Link naming follows wheel_module.xacro: wheel_{position}_link / steering_{position}_link
+  -->
+  <xacro:macro name="WheelFriction" params="position">
+    <gazebo reference="wheel_${position}_link">
       <mu1>1.8</mu1>
       <mu2>1.8</mu2>
@@ -15,13 +17,13 @@
       <minDepth>0.001</minDepth>
     </gazebo>
-    <gazebo reference="${prefix}_steering_link">
+    <gazebo reference="steering_${position}_link">
       <mu1>0.0</mu1>
       <mu2>0.0</mu2>
     </gazebo>
   </xacro:macro>
-  <xacro:WheelFriction prefix="front_left"/>
-  <xacro:WheelFriction prefix="front_right"/>
-  <xacro:WheelFriction prefix="rear_left"/>
-  <xacro:WheelFriction prefix="rear_right"/>
+  <xacro:WheelFriction position="front_left"/>
+  <xacro:WheelFriction position="front_right"/>
+  <xacro:WheelFriction position="rear_left"/>
+  <xacro:WheelFriction position="rear_right"/>
   <!-- ── ign_ros2_control plugin ── -->
   <gazebo>
